Commit message: [MultiversePlayer] picking up works

File: resources/multiverse_episodes/icub_montessori_no_hands/models/montessori_object_1.urdf (robot description, URDF)
Before this commit: robot montessori_object_1, 2 links, 1 joints
Links:
- removed link world
Joints:
- removed joint montessori_object_1_joint

File: resources/multiverse_episodes/icub_montessori_no_hands/models/montessori_object_2.urdf (robot description, URDF)
Before this commit: robot montessori_object_2, 2 links, 1 joints
Links:
- removed link world
Joints:
- removed joint montessori_object_2_joint

File: resources/multiverse_episodes/icub_montessori_no_hands/models/montessori_object_3.urdf (robot description, URDF)
Before this commit: robot montessori_object_3, 2 links, 1 joints
Links:
- removed link world
Joints:
- removed joint montessori_object_3_joint

File: resources/multiverse_episodes/icub_montessori_no_hands/models/montessori_object_4.urdf (robot description, URDF)
Before this commit: robot montessori_object_4, 2 links, 1 joints
Links:
- removed link world
Joints:
- removed joint montessori_object_4_joint

File: resources/multiverse_episodes/icub_montessori_no_hands/models/montessori_object_5.urdf (robot description, URDF)
Before this commit: robot montessori_object_5, 2 links, 1 joints
Links:
- removed link world
Joints:
- removed joint montessori_object_5_joint

File: resources/multiverse_episodes/icub_montessori_no_hands/models/montessori_object_6.urdf (robot description, URDF)
Before this commit: robot montessori_object_6, 2 links, 1 joints
Links:
- removed link montessori_object_5
Joints:
- removed joint montessori_object_6_joint

File: resources/multiverse_episodes/icub_montessori_no_hands/models/scene.urdf (robot description, URDF)
Before this commit: robot iCub_with_montessori_toys_2, 125 links, 124 joints
Links:
- removed link base_footprint
- removed link base_link
- removed link chest
- removed link chest_depth_frame
- removed link chest_rgb_frame
- removed link eyes_tilt_frame
- removed link head
- removed link iCub
- removed link imu_frame
- removed link l_ankle_1
- removed link l_ankle_2
- removed link l_elbow_1
- removed link l_eye
- removed link l_foot_front
- removed link l_foot_rear
- removed link l_forearm
- removed link l_gripper_tool_frame
- removed link l_hand
- removed link l_hand_index_0
- removed link l_hand_index_1
- removed link l_hand_index_2
- removed link l_hand_index_3
- removed link l_hand_index_tip
- removed link l_hand_little_0
- removed link l_hand_little_1
- removed link l_hand_little_2
- removed link l_hand_little_3
- removed link l_hand_little_tip
- removed link l_hand_middle_0
- removed link l_hand_middle_1
- removed link l_hand_middle_2
- removed link l_hand_middle_3
- removed link l_hand_middle_tip
- removed link l_hand_ring_0
- removed link l_hand_ring_1
- removed link l_hand_ring_2
- removed link l_hand_ring_3
- removed link l_hand_ring_tip
- removed link l_hand_thumb_0
- removed link l_hand_thumb_1
- removed link l_hand_thumb_2
- removed link l_hand_thumb_3
- removed link l_hand_thumb_tip
- removed link l_hip_1
- removed link l_hip_2
- removed link l_hip_3
- removed link l_lower_leg
- removed link l_shoulder_1
- removed link l_shoulder_2
- removed link l_shoulder_3
- removed link l_sole
- removed link l_upper_arm
- removed link l_upper_leg
- removed link l_wrist_1
- removed link montessori_object_1
- removed link montessori_object_2
- removed link montessori_object_2_ref
- removed link montessori_object_3
- removed link montessori_object_3_ref
- removed link montessori_object_4
- removed link montessori_object_5
- removed link montessori_object_5_ref
- removed link montessori_object_6
- removed link montessori_object_6_ref
- removed link neck_1
- removed link neck_2
- removed link neck_3
- removed link r_ankle_1
- removed link r_ankle_2
- removed link r_elbow_1
- removed link r_eye
- removed link r_foot_front
- removed link r_foot_rear
- removed link r_forearm
- removed link r_gripper_tool_frame
- removed link r_hand
- removed link r_hand_index_0
- removed link r_hand_index_1
- removed link r_hand_index_2
- removed link r_hand_index_3
- removed link r_hand_index_tip
- removed link r_hand_little_0
- removed link r_hand_little_1
- removed link r_hand_little_2
- removed link r_hand_little_3
- removed link r_hand_little_tip
- removed link r_hand_middle_0
- removed link r_hand_middle_1
- removed link r_hand_middle_2
- removed link r_hand_middle_3
- removed link r_hand_middle_tip
- removed link r_hand_ring_0
- removed link r_hand_ring_1
- removed link r_hand_ring_2
- removed link r_hand_ring_3
- removed link r_hand_ring_tip
- removed link r_hand_thumb_0
- removed link r_hand_thumb_1
- removed link r_hand_thumb_2
- removed link r_hand_thumb_3
- removed link r_hand_thumb_tip
- removed link r_hip_1
- removed link r_hip_2
- removed link r_hip_3
- removed link r_lower_leg
- removed link r_shoulder_1
- removed link r_shoulder_2
- removed link r_shoulder_3
- removed link r_sole
- removed link r_upper_arm
- removed link r_upper_leg
- removed link r_wrist_1
- removed link root_link
- removed link torso_1
- removed link torso_2
Joints:
- removed joint base_footprint_joint
- removed joint base_link_joint
- removed joint chest_depth_frame_joint
- removed joint chest_rgb_frame_joint
- removed joint eyes_tilt
- removed joint iCub_joint
- removed joint imu_frame_joint
- removed joint l_ankle_pitch
- removed joint l_ankle_roll
- removed joint l_elbow
- removed joint l_eye_pan_joint
- removed joint l_foot_front_joint
- removed joint l_foot_rear_joint
- removed joint l_gripper_tool_frame_joint
- removed joint l_hand_index_0_joint
- removed joint l_hand_index_1_joint
- removed joint l_hand_index_2_joint
- removed joint l_hand_index_3_joint
- removed joint l_hand_index_tip_joint
- removed joint l_hand_little_0_joint
- removed joint l_hand_little_1_joint
- removed joint l_hand_little_2_joint
- removed joint l_hand_little_3_joint
- removed joint l_hand_little_tip_joint
- removed joint l_hand_middle_0_joint
- removed joint l_hand_middle_1_joint
- removed joint l_hand_middle_2_joint
- removed joint l_hand_middle_3_joint
- removed joint l_hand_middle_tip_joint
- removed joint l_hand_ring_0_joint
- removed joint l_hand_ring_1_joint
- removed joint l_hand_ring_2_joint
- removed joint l_hand_ring_3_joint
- removed joint l_hand_ring_tip_joint
- removed joint l_hand_thumb_0_joint
- removed joint l_hand_thumb_1_joint
- removed joint l_hand_thumb_2_joint
- removed joint l_hand_thumb_3_joint
- removed joint l_hand_thumb_tip_joint
- removed joint l_hip_3_joint
- removed joint l_hip_pitch
- removed joint l_hip_roll
- removed joint l_hip_yaw
- removed joint l_knee
- removed joint l_shoulder_3_joint
- removed joint l_shoulder_pitch
- removed joint l_shoulder_roll
- removed joint l_shoulder_yaw
- removed joint l_sole_joint
- removed joint l_wrist_pitch
- removed joint l_wrist_prosup
- removed joint l_wrist_yaw
- removed joint montessori_object_1_joint
- removed joint montessori_object_2_joint
- removed joint montessori_object_2_ref_joint
- removed joint montessori_object_3_joint
- removed joint montessori_object_3_ref_joint
- removed joint montessori_object_4_joint
- removed joint montessori_object_5_joint
- removed joint montessori_object_5_ref_joint
- removed joint montessori_object_6_joint
- removed joint montessori_object_6_ref_joint
- removed joint neck_1_joint
- removed joint neck_pitch
- removed joint neck_roll
- removed joint neck_yaw
- removed joint r_ankle_pitch
- removed joint r_ankle_roll
- removed joint r_elbow
- removed joint r_eye_pan_joint
- removed joint r_foot_front_joint
- removed joint r_foot_rear_joint
- removed joint r_gripper_tool_frame_joint
- removed joint r_hand_index_0_joint
- removed joint r_hand_index_1_joint
- removed joint r_hand_index_2_joint
- removed joint r_hand_index_3_joint
- removed joint r_hand_index_tip_joint
- removed joint r_hand_little_0_joint
- removed joint r_hand_little_1_joint
- removed joint r_hand_little_2_joint
- removed joint r_hand_little_3_joint
- removed joint r_hand_little_tip_joint
- removed joint r_hand_middle_0_joint
- removed joint r_hand_middle_1_joint
- removed joint r_hand_middle_2_joint
- removed joint r_hand_middle_3_joint
- removed joint r_hand_middle_tip_joint
- removed joint r_hand_ring_0_joint
- removed joint r_hand_ring_1_joint
- removed joint r_hand_ring_2_joint
- removed joint r_hand_ring_3_joint
- removed joint r_hand_ring_tip_joint
- removed joint r_hand_thumb_0_joint
- removed joint r_hand_thumb_1_joint
- removed joint r_hand_thumb_2_joint
- removed joint r_hand_thumb_3_joint
- removed joint r_hand_thumb_tip_joint
- removed joint r_hip_3_joint
- removed joint r_hip_pitch
- removed joint r_hip_roll
- removed joint r_hip_yaw
- removed joint r_knee
- removed joint r_shoulder_3_joint
- removed joint r_shoulder_pitch
- removed joint r_shoulder_roll
- removed joint r_shoulder_yaw
- removed joint r_sole_joint
- removed joint r_wrist_pitch
- removed joint r_wrist_prosup
- removed joint r_wrist_yaw
- removed joint root_link_joint
- removed joint torso_pitch
- removed joint torso_roll
- removed joint torso_yaw
