Commit message: [Segmind] added virtual links to shaped holes.

File: resources/multiverse_episodes/icub_montessori_no_hands/models/scene.urdf (robot description, URDF)
Before this commit: robot iCub_with_montessori_toys_2, 10 links, 9 joints
Links:
- added link circular_hole_1, mass 0.007762390188872814; visual cylinder length=0.01 radius=0.015
- added link circular_hole_2, mass 0.007762390188872814; visual cylinder length=0.01 radius=0.02
- added link rectangular_hole, mass 0.008732689544558525; visual box size=0.019999999552965164 0.03999999910593033 0.0299999993294477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
- added link square_hole, mass 0.007762390188872814; visual box size=0.03 0.03 0.03
- added link triangle_hole, mass 0.01134410034865141; visual mesh filename=file://montessori_object_1/meshes/stl/montessori_object_2_M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 scale=1.0 1.0 1.0
Joints:
- added joint montessori_circular_hole_1_joint: type fixed, parent montessori_box, child circular_hole_1, origin xyz=-0.0215 -0.087 0.035 rpy=0.0 0.0 0.0
- added joint montessori_circular_hole_2_joint: type fixed, parent montessori_box, child circular_hole_2, origin xyz=-0.018 0.091 0.035 rpy=0.0 0.0 0.0
- added joint montessori_rectangular_hole_joint: type fixed, parent montessori_box, child rectangular_hole, origin xyz=-0.027 0.0 0.035 rpy=0.0 0.0 0.0
- added joint montessori_square_hole_joint: type fixed, parent montessori_box, child square_hole, origin xyz=0.02 -0.087 0.035 rpy=0.0 0.0 0.0
- added joint montessori_triangle_hole_joint: type fixed, parent montessori_box, child triangle_hole, origin xyz=0.019 0.0 0.035 rpy=0.0 0.0 0.0

Commit message: [Segmind] collision detecting virtual link holes.

File: resources/multiverse_episodes/icub_montessori_no_hands/models/scene.urdf (robot description, URDF)
Before this commit: robot iCub_with_montessori_toys_2, 15 links, 14 joints
Links:
- link circular_hole_1: geometry collision cylinder length=0.01 radius=0.015
- link circular_hole_2: geometry collision cylinder length=0.01 radius=0.02
- link rectangular_hole: geometry collision box size=0.019999999552965164 0.03999999910593033 0.0299999993294477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
- link square_hole: geometry collision box size=0.03 0.03 0.03
- link triangle_hole: geometry collision mesh filename=file://montessori_object_1/meshes/stl/montessori_object_2_M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 scale=1.0 1.0 1.0

Commit message: [Segmind] insertion with hole detection works.

File: resources/multiverse_episodes/icub_montessori_no_hands/models/scene.urdf (robot description, URDF)
Before this commit: robot iCub_with_montessori_toys_2, 15 links, 14 joints
Links:
- link circular_hole_1: geometry collision cylinder length=0.025 radius=0.019
- link circular_hole_2: geometry collision cylinder length=0.025 radius=0.024
- link rectangular_hole: geometry collision box size=0.023 0.043 0.033
- link square_hole: geometry collision box size=0.036 0.036 0.036
- link triangle_hole: geometry collision mesh filename=file://montessori_object_1/meshes/stl/montessori_object_2_M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 scale=1.2 1.2 1.2

Commit message: [IcubDemo] fully works.

File: resources/multiverse_episodes/icub_montessori_no_hands/models/scene.urdf (robot description, URDF)
Before this commit: robot iCub_with_montessori_toys_2, 15 links, 14 joints
Links:
- link circular_hole_1: geometry collision cylinder length=0.025 radius=0.017
- link circular_hole_2: geometry collision cylinder length=0.025 radius=0.022
- link rectangular_hole: geometry collision box size=0.02 0.04 0.03
- link square_hole: geometry collision box size=0.03 0.03 0.03
- link triangle_hole: geometry collision mesh filename=file://montessori_object_1/meshes/stl/montessori_object_2_M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 scale=1.1 1.1 1.1
Joints:
- joint montessori_circular_hole_1_joint: origin xyz=-0.0215 -0.087 0.035 rpy=0.0 0.0 0.0 -> xyz=-0.0215 -0.087 0.03 rpy=0.0 0.0 0.0
- joint montessori_circular_hole_2_joint: origin xyz=-0.018 0.091 0.035 rpy=0.0 0.0 0.0 -> xyz=-0.018 0.091 0.03 rpy=0.0 0.0 0.0
- joint montessori_rectangular_hole_joint: origin xyz=-0.027 0.0 0.035 rpy=0.0 0.0 0.0 -> xyz=-0.027 0.0 0.025 rpy=0.0 0.0 0.0
- joint montessori_square_hole_joint: origin xyz=0.02 -0.087 0.035 rpy=0.0 0.0 0.0 -> xyz=0.02 -0.087 0.03 rpy=0.0 0.0 0.0
- joint montessori_triangle_hole_joint: origin xyz=0.019 0.0 0.035 rpy=0.0 0.0 0.0 -> xyz=0.019 0.0 0.03 rpy=0.0 0.0 0.0

Commit message: [Segmind] update to insertion, docker, and scene

File: resources/multiverse_episodes/icub_montessori_no_hands/models/scene.urdf (robot description, URDF)
Before this commit: robot iCub_with_montessori_toys_2, 15 links, 14 joints
Joints:
- joint montessori_box_joint: type floating -> fixed
- joint small_table_joint: type floating -> fixed
- joint table_joint: type floating -> fixed

Commit message: [IcubDemo] tuned hole sizes in urdf, and detector running frequency.

File: resources/multiverse_episodes/icub_montessori_no_hands/models/scene.urdf (robot description, URDF)
Before this commit: robot iCub_with_montessori_toys_2, 15 links, 14 joints
Links:
- link circular_hole_1: geometry collision cylinder length=0.01 radius=0.017
- link circular_hole_2: geometry collision cylinder length=0.01 radius=0.022
- link rectangular_hole: geometry collision box size=0.02 0.04 0.01
- link square_hole: geometry collision box size=0.03 0.03 0.005
- link triangle_hole: geometry collision mesh filename=file://montessori_object_1/meshes/stl/montessori_object_2_M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 scale=1.1 1.1 0.3

Commit message: [IcubDemo] demo fixes

File: resources/multiverse_episodes/icub_montessori_no_hands/models/scene.urdf (robot description, URDF)
Before this commit: robot iCub_with_montessori_toys_2, 15 links, 14 joints
Links:
- link circular_hole_1: geometry collision cylinder length=0.005 radius=0.019
- link rectangular_hole: geometry collision box size=0.02 0.04 0.005
Joints:
- joint montessori_rectangular_hole_joint: origin xyz=-0.027 0.0 0.025 rpy=0.0 0.0 0.0 -> xyz=-0.027 0.0 0.035 rpy=0.0 0.0 0.0

Commit message: [IcubDemo] continuous running demo.

File: resources/multiverse_episodes/icub_montessori_no_hands/models/scene.urdf (robot description, URDF)
Before this commit: robot iCub_with_montessori_toys_2, 15 links, 14 joints
Joints:
- joint montessori_circular_hole_1_joint: origin xyz=-0.0215 -0.087 0.03 rpy=0.0 0.0 0.0 -> xyz=-0.0215 -0.087 0.025 rpy=0.0 0.0 0.0
- joint montessori_circular_hole_2_joint: origin xyz=-0.018 0.091 0.03 rpy=0.0 0.0 0.0 -> xyz=-0.018 0.091 0.025 rpy=0.0 0.0 0.0
- joint montessori_rectangular_hole_joint: origin xyz=-0.027 0.0 0.035 rpy=0.0 0.0 0.0 -> xyz=-0.027 0.0 0.03 rpy=0.0 0.0 0.0
- joint montessori_triangle_hole_joint: origin xyz=0.019 0.0 0.03 rpy=0.0 0.0 0.0 -> xyz=0.019 0.0 0.025 rpy=0.0 0.0 0.0

Commit message: [IcubDemo] demo updates

File: resources/multiverse_episodes/icub_montessori_no_hands/models/scene.urdf (robot description, URDF)
Before this commit: robot iCub_with_montessori_toys_2, 15 links, 14 joints
Joints:
- joint montessori_circular_hole_1_joint: origin xyz=-0.0215 -0.087 0.025 rpy=0.0 0.0 0.0 -> xyz=-0.0215 -0.087 0.017 rpy=0.0 0.0 0.0
- joint montessori_circular_hole_2_joint: origin xyz=-0.018 0.091 0.025 rpy=0.0 0.0 0.0 -> xyz=-0.018 0.091 0.02 rpy=0.0 0.0 0.0
- joint montessori_rectangular_hole_joint: origin xyz=-0.027 0.0 0.03 rpy=0.0 0.0 0.0 -> xyz=-0.027 0.0 0.02 rpy=0.0 0.0 0.0
- joint montessori_square_hole_joint: origin xyz=0.02 -0.087 0.03 rpy=0.0 0.0 0.0 -> xyz=0.02 -0.087 0.02 rpy=0.0 0.0 0.0
- joint montessori_triangle_hole_joint: origin xyz=0.019 0.0 0.025 rpy=0.0 0.0 0.0 -> xyz=0.019 0.0 0.02 rpy=0.0 0.0 0.0

Commit message: [IcubDemo] better insertion, added shape matching phase, corrected pose problems.

File: resources/multiverse_episodes/icub_montessori_no_hands/models/scene.urdf (robot description, URDF)
Before this commit: robot iCub_with_montessori_toys_2, 15 links, 14 joints
Joints:
- joint montessori_circular_hole_1_joint: origin xyz=-0.0215 -0.087 0.017 rpy=0.0 0.0 0.0 -> xyz=-0.0215 -0.087 0.025 rpy=0.0 0.0 0.0
- joint montessori_circular_hole_2_joint: origin xyz=-0.018 0.091 0.02 rpy=0.0 0.0 0.0 -> xyz=-0.018 0.091 0.025 rpy=0.0 0.0 0.0
- joint montessori_rectangular_hole_joint: origin xyz=-0.027 0.0 0.02 rpy=0.0 0.0 0.0 -> xyz=-0.027 0.0 0.025 rpy=0.0 0.0 0.0
- joint montessori_square_hole_joint: origin xyz=0.02 -0.087 0.02 rpy=0.0 0.0 0.0 -> xyz=0.02 -0.087 0.025 rpy=0.0 0.0 0.0
- joint montessori_triangle_hole_joint: origin xyz=0.019 0.0 0.02 rpy=0.0 0.0 0.0 -> xyz=0.019 0.0 0.025 rpy=0.0 0.0 0.0

Commit message: [IcubDemo] demo updates

File: resources/multiverse_episodes/icub_montessori_no_hands/models/scene.urdf (robot description, URDF)
Before this commit: robot iCub_with_montessori_toys_2, 15 links, 14 joints
Links:
- added link disk_hole, mass 0.007762390188872814; collision box size=0.01 0.03 0.001
- link circular_hole_1: geometry collision cylinder length=0.001 radius=0.015
- link circular_hole_2: geometry collision cylinder length=0.001 radius=0.015
- link rectangular_hole: geometry collision box size=0.015 0.03 0.001
- link square_hole: geometry collision box size=0.025 0.025 0.001
- link triangle_hole: geometry collision mesh filename=file://montessori_object_1/meshes/stl/montessori_object_2_M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 scale=0.8 0.8 0.1
Joints:
- added joint montessori_disk_hole_joint: type fixed, parent montessori_box, child disk_hole, origin xyz=-0.018 0.091 0.04 rpy=0.0 0.0 0.0
- joint montessori_circular_hole_1_joint: origin xyz=-0.0215 -0.087 0.025 rpy=0.0 0.0 0.0 -> xyz=-0.0215 -0.087 0.04 rpy=0.0 0.0 0.0
- joint montessori_circular_hole_2_joint: origin xyz=-0.018 0.091 0.025 rpy=0.0 0.0 0.0 -> xyz=-0.018 0.091 0.04 rpy=0.0 0.0 0.0
- joint montessori_rectangular_hole_joint: origin xyz=-0.027 0.0 0.025 rpy=0.0 0.0 0.0 -> xyz=-0.027 0.0 0.04 rpy=0.0 0.0 0.0
- joint montessori_square_hole_joint: origin xyz=0.02 -0.087 0.025 rpy=0.0 0.0 0.0 -> xyz=0.02 -0.087 0.04 rpy=0.0 0.0 0.0
- joint montessori_triangle_hole_joint: origin xyz=0.019 0.0 0.025 rpy=0.0 0.0 0.0 -> xyz=0.019 0.0 0.04 rpy=0.0 0.0 0.0

Commit message: [IcubDemo] demo updates

File: resources/multiverse_episodes/icub_montessori_no_hands/models/scene.urdf (robot description, URDF)
Before this commit: robot iCub_with_montessori_toys_2, 16 links, 15 joints
Links:
- link small_table: geometry collision box size=0.05000000074505806 0.05000000074505806 0.25; collision box size=0.05000000074505806 0.05000000074505806 0.25
Joints:
- joint montessori_box_joint: origin xyz=-0.4 0.0 1.39 rpy=0.0 0.0 0.0 -> xyz=-0.4 0.0 1.353 rpy=0.0 0.0 0.0
- joint small_table_joint: origin xyz=-0.35 0.0 1.0 rpy=0.0 0.0 0.0 -> xyz=-0.35 0.0 1.05 rpy=0.0 0.0 0.0

Commit message: [IcubDemo] demo updates

File: resources/multiverse_episodes/icub_montessori_no_hands/models/scene.urdf (robot description, URDF)
Before this commit: robot iCub_with_montessori_toys_2, 16 links, 15 joints
Links:
- link triangle_hole: geometry collision mesh filename=file://montessori_object_1/meshes/stl/montessori_object_2_M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 scale=0.8 0.8 0.05

Commit message: [IcubDemo] demo updates

File: resources/multiverse_episodes/icub_montessori_no_hands/models/scene.urdf (robot description, URDF)
Before this commit: robot iCub_with_montessori_toys_2, 16 links, 15 joints
Links:
- link triangle_hole: geometry collision mesh filename=file://montessori_object_1/meshes/stl/montessori_object_2_M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 scale=0.8 0.8 0.02

Commit message: [IcubDemo] demo updates

File: resources/multiverse_episodes/icub_montessori_no_hands/models/scene.urdf (robot description, URDF)
Before this commit: robot iCub_with_montessori_toys_2, 16 links, 15 joints
Links:
- link square_hole: geometry collision box size=0.03 0.03 0.001

Commit message: [IcubDemo] demo fixes.

File: resources/multiverse_episodes/icub_montessori_no_hands/models/scene.urdf (robot description, URDF)
Before this commit: robot iCub_with_montessori_toys_2, 16 links, 15 joints
Links:
- link disk_hole: geometry collision box size=0.005 0.04 0.001
Joints:
- joint montessori_disk_hole_joint: origin xyz=-0.018 0.091 0.04 rpy=0.0 0.0 0.0 -> xyz=0.025 0.091 0.04 rpy=0.0 0.0 0.0
